Commit message: fixed frames to match DH

File: robotics_description/urdf/p1.xacro (robot description, xacro)
@@ -24,4 +24,5 @@
     <link name="base_link">
         <visual>
+            <origin xyz="0 0 0" rpy="0 0 0 "/>
             <geometry>
                 <cylinder radius="0.10" length="0.01"/>
@@ -54,5 +55,5 @@
     <link name="link2">
         <visual>
-            <origin xyz="0 0.25 0.0" rpy="${pi/2} 0 0 "/>
+            <origin xyz="0.25 0 0.0" rpy="${pi/2} 0 ${-pi/2}  "/>
             <geometry>
                 <cylinder radius="0.02" length="0.5"/>
@@ -70,15 +71,15 @@
     <link name="link3">
         <visual>
+            <origin xyz="0 0 0.25" rpy="${pi} 0 0"/>
+            <geometry>
+                <cylinder radius="0.02" length="0.5"/>
+            </geometry>
+            <material name="blue"/>
+        </visual>
+        <collision>
             <origin xyz="0 0.25 0" rpy="${pi/2} 0 0"/>
             <geometry>
                 <cylinder radius="0.02" length="0.5"/>
             </geometry>
-            <material name="blue"/>
-        </visual>
-        <collision>
-            <origin xyz="0 0.25 0" rpy="${pi/2} 0 0"/>
-            <geometry>
-                <cylinder radius="0.02" length="0.5"/>
-            </geometry>
         </collision>
         <xacro:default_inertial mass="1"/>
@@ -86,6 +87,7 @@
     <link name="link4">
         <visual>
-            <geometry>
-                <box size="0.08 0.08 0.08"/>
+            <origin xyz="0 0 0.10" rpy="${pi/2} ${pi} 0"/>
+            <geometry>
+                <mesh filename="package://robotics/robotics_description/meshes/spoon.stl" scale="0.003 0.003 0.003"/>
             </geometry>
             <material name="black"/>
@@ -93,5 +95,5 @@
         <collision>
             <geometry>
-                <box size="0.08 0.08 0.08"/>
+                <mesh filename="package://robotics/robotics_description/meshes/spoon.stl" scale="0.003 0.003 0.003"/>
             </geometry>
         </collision>
@@ -117,8 +119,9 @@
     <joint name="joint5" type="fixed">
         <origin xyz="0 0 0" rpy="0 0 0"/>
-        <parent link="base_link"/>
+        <parent link="dummy"/>
         <child link="link5"/>
     </joint>
     <joint name="dummy_joint" type="fixed">
+        <origin xyz="0 0 0" rpy="0 0 0"/>
         <parent link="dummy"/>
         <child link="base_link"/>
@@ -139,12 +142,12 @@
     </joint>
     <joint name="joint3" type="revolute">
-        <origin xyz="0 0.5 0." rpy="${pi/2} 0 ${pi/2}"/>
+        <origin xyz="0.5 0 0." rpy="${pi} 0 ${-pi/2}"/>
         <parent link="link2"/>
         <child link="link3"/>
         <axis xyz="0 0 1"/>
-        <limit lower="${-3*pi/2}" upper="${-pi/2}" effort="50" velocity="1"/>
+        <limit lower="${-pi}" upper="${pi}" effort="50" velocity="1"/>
     </joint>
     <joint name="joint4" type="revolute">
-        <origin xyz="0 0.5 0" rpy="${-pi/2} 0 0"/>
+        <origin xyz="0 0 0.5" rpy="${pi/2} 0 ${pi}"/>
         <parent link="link3"/>
         <child link="link4"/>

Commit message: Actually follows DH now

File: robotics_description/urdf/p1.xacro (robot description, xacro)
@@ -71,5 +71,5 @@
     <link name="link3">
         <visual>
-            <origin xyz="0 0 0.25" rpy="${pi} 0 0"/>
+            <origin xyz="0.25 0 0" rpy="${pi/2} 0 ${pi/2}"/>
             <geometry>
                 <cylinder radius="0.02" length="0.5"/>
@@ -87,5 +87,5 @@
     <link name="link4">
         <visual>
-            <origin xyz="0 0 0.10" rpy="${pi/2} ${pi} 0"/>
+            <origin xyz="0 0 -0.125" rpy="${pi/2} ${pi} 0"/>
             <geometry>
                 <mesh filename="package://robotics/robotics_description/meshes/spoon.stl" scale="0.003 0.003 0.003"/>
@@ -139,19 +139,19 @@
         <child link="link2"/>
         <axis xyz="0 0 1"/>
-        <limit lower="${-pi/2}" upper="${pi/2}" effort="50" velocity="1"/>
+        <limit lower="${-2*pi}" upper="${2*pi}" effort="50" velocity="1"/>
     </joint>
     <joint name="joint3" type="revolute">
-        <origin xyz="0.5 0 0." rpy="${pi} 0 ${-pi/2}"/>
+        <origin xyz="0.5 0 0." rpy="${pi/2} 0 0"/>
         <parent link="link2"/>
         <child link="link3"/>
         <axis xyz="0 0 1"/>
-        <limit lower="${-pi}" upper="${pi}" effort="50" velocity="1"/>
+        <limit lower="${-2*pi}" upper="${2*pi}" effort="50" velocity="1"/>
     </joint>
     <joint name="joint4" type="revolute">
-        <origin xyz="0 0 0.5" rpy="${pi/2} 0 ${pi}"/>
+        <origin xyz="0.50 0 0.25" rpy="0 0 0"/>
         <parent link="link3"/>
         <child link="link4"/>
         <axis xyz="0 0 1"/>
-        <limit lower="${-pi/2}" upper="${pi/2}" effort="50" velocity="1"/>
+        <limit lower="${-2*pi}" upper="${2*pi}" effort="50" velocity="1"/>
     </joint>
     <!--TRANS STUFF-->
