Commit message: NEW DIRECTORYIES FOR NEW PROJECTS and working forward kinamatics

File: projects/p1/p1_description/urdf/p1.xacro (robot description, xacro)
@@ -89,5 +89,5 @@
             <origin xyz="0 0 -0.125" rpy="${pi/2} ${pi} 0"/>
             <geometry>
-                <mesh filename="package://robotics/robotics_description/meshes/spoon.stl" scale="0.003 0.003 0.003"/>
+                <mesh filename="package://robotics/projects/p1/p1_description/meshes/spoon.stl" scale="0.003 0.003 0.003"/>
             </geometry>
             <material name="black"/>
@@ -95,5 +95,5 @@
         <collision>
             <geometry>
-                <mesh filename="package://robotics/robotics_description/meshes/spoon.stl" scale="0.003 0.003 0.003"/>
+                <mesh filename="package://robotics/projects/p1/p1_description/meshes/spoon.stl" scale="0.003 0.003 0.003"/>
             </geometry>
         </collision>
@@ -197,4 +197,4 @@
         </plugin>
     </gazebo>
-    <xacro:include filename="$(find robotics)/robotics_description/urdf/p1.gazebo" />
+    <xacro:include filename="$(find robotics)/projects/p1/p1_description/urdf/p1.gazebo" />
 </robot>
